Commit message: init

File: my_robot_description/urdf/Final.urdf.xacro (robot description, xacro)
@@ -344,5 +344,5 @@
         <mesh filename="package://my_robot_description/meshes/link3.STL" />
       </geometry>
-      <material name="yellow "/>
+      <material name="yellow"/>
     </visual>
     <collision>

File: my_robot_description/urdf/gazebo_plugin.xacro (robot description, xacro)
@@ -13,5 +13,5 @@
             <odom_topic>odom</odom_topic>
             <tf_topic>tf</tf_topic>
-            <publish_odom_tf>true</publish_odom_tf>
+            <publish_odom_tf>false</publish_odom_tf>
             <frame_id>odom</frame_id>
             <child_frame_id>base_footprint</child_frame_id>
@@ -65,5 +65,5 @@
     <gazebo reference="lidar">
         <sensor name="lidar_sensor" type="gpu_lidar"> <always_on>true</always_on>
-            <visualize>true</visualize> <update_rate>10.0</update_rate>
+            <visualize>true</visualize> <update_rate>20.0</update_rate>
             <topic>scan</topic>
             <ignition_frame_id>lidar</ignition_frame_id>
@@ -79,5 +79,5 @@
                 <range>
                     <min>0.15</min>
-                    <max>12.0</max>
+                    <max>25.0</max>
                     <resolution>0.01</resolution>
                 </range>
@@ -116,20 +116,17 @@
             <update_rate>100</update_rate>
             <visualize>true</visualize>
-            <plugin filename="libgazebo_ros_imu_sensor.so" name="imu_plugin">
-                <ros>
-                <remapping>~/out:=imu</remapping>
-                </ros>
-                <initial_orientation_as_reference>false</initial_orientation_as_reference>
-            </plugin>
+            <!-- CHỈ DÙNG 2 DÒNG NÀY ĐỂ ĐỊNH NGHĨA TOPIC VÀ FRAME CHO IGNITION -->
+            <topic>imu</topic>
+            <ignition_frame_id>imu</ignition_frame_id>
             <imu>
                 <angular_velocity>
-                <x><noise type="gaussian"><mean>0.0</mean><stddev>2e-4</stddev></noise></x>
-                <y><noise type="gaussian"><mean>0.0</mean><stddev>2e-4</stddev></noise></y>
-                <z><noise type="gaussian"><mean>0.0</mean><stddev>2e-4</stddev></noise></z>
+                    <x><noise type="gaussian"><mean>0.0</mean><stddev>2e-4</stddev></noise></x>
+                    <y><noise type="gaussian"><mean>0.0</mean><stddev>2e-4</stddev></noise></y>
+                    <z><noise type="gaussian"><mean>0.0</mean><stddev>2e-4</stddev></noise></z>
                 </angular_velocity>
                 <linear_acceleration>
-                <x><noise type="gaussian"><mean>0.0</mean><stddev>1.7e-2</stddev></noise></x>
-                <y><noise type="gaussian"><mean>0.0</mean><stddev>1.7e-2</stddev></noise></y>
-                <z><noise type="gaussian"><mean>0.0</mean><stddev>1.7e-2</stddev></noise></z>
+                    <x><noise type="gaussian"><mean>0.0</mean><stddev>1.7e-2</stddev></noise></x>
+                    <y><noise type="gaussian"><mean>0.0</mean><stddev>1.7e-2</stddev></noise></y>
+                    <z><noise type="gaussian"><mean>0.0</mean><stddev>1.7e-2</stddev></noise></z>
                 </linear_acceleration>
             </imu>
@@ -152,5 +149,5 @@
         <mu2>0.0</mu2>
     </gazebo>
-    <gazebo reference="wheel_left">
+    <!-- <gazebo reference="wheel_left">
         <mu1>200.0</mu1>
         <mu2>100.0</mu2>
@@ -159,4 +156,4 @@
         <mu1>200.0</mu1>
         <mu2>100.0</mu2>
-    </gazebo>
+    </gazebo> -->
 </robot>

Commit message: https://github.com/TNSang25/ROS2-cuoi-ki.git

File: my_robot_description/urdf/Final.urdf.xacro (robot description, xacro)
@@ -358,5 +358,5 @@
     <child link="link3" />
     <axis xyz="0 0 1" />
-    <limit lower="-3.14" upper="3.14" effort="100" velocity="100" />
+    <limit lower="-3.14" upper="3.14" effort="0" velocity="0" />
   </joint>
   <link name="ef"></link>

File: my_robot_description/urdf/gazebo_plugin.xacro (robot description, xacro)
@@ -10,8 +10,8 @@
             <wheel_radius>0.07</wheel_radius>
             <odom_publish_frequency>50</odom_publish_frequency>
-            <topic>cmd_vel</topic>
+            <topic>/cmd_vel</topic>
             <odom_topic>odom</odom_topic>
             <tf_topic>tf</tf_topic>
-            <publish_odom_tf>false</publish_odom_tf>
+            <publish_odom_tf>true</publish_odom_tf>
             <frame_id>odom</frame_id>
             <child_frame_id>base_footprint</child_frame_id>
@@ -78,6 +78,6 @@
                 </scan>
                 <range>
-                    <min>0.15</min>
-                    <max>25.0</max>
+                    <min>0.01</min>
+                    <max>20.0</max>
                     <resolution>0.01</resolution>
                 </range>
@@ -134,26 +134,18 @@
     </gazebo>
     <gazebo reference="mat_trau1">
-        <mu1>0.0</mu1>
-        <mu2>0.0</mu2>
+        <mu1>0.01</mu1>
+        <mu2>0.01</mu2>
     </gazebo>
     <gazebo reference="mat_trau2">
-        <mu1>0.0</mu1>
-        <mu2>0.0</mu2>
+        <mu1>0.01</mu1>
+        <mu2>0.01</mu2>
     </gazebo>
     <gazebo reference="mat_trau3">
-        <mu1>0.0</mu1>
-        <mu2>0.0</mu2>
+        <mu1>0.01</mu1>
+        <mu2>0.01</mu2>
     </gazebo>
     <gazebo reference="mat_trau4">
-        <mu1>0.0</mu1>
-        <mu2>0.0</mu2>
+        <mu1>0.01</mu1>
+        <mu2>0.01</mu2>
     </gazebo>
-    <!-- <gazebo reference="wheel_left">
-        <mu1>200.0</mu1>
-        <mu2>100.0</mu2>
-    </gazebo>
-    <gazebo reference="wheel_right">
-        <mu1>200.0</mu1>
-        <mu2>100.0</mu2>
-    </gazebo> -->
 </robot>
